Commit message: Added bubble at each joint and EE. TODO: self-collision

File: src/scripts/panda_spart/panda.urdf (robot description, URDF)
Before this commit: robot kuka_lwr, 8 links, 7 joints
Links:
- added link panda_ee, mass 0; collision mesh filename=meshes_panda/link7.obj
Joints:
- added joint panda_joint8: type revolute, parent panda_link7, child panda_ee, origin xyz=0 0 0.1070 rpy=0 0 0, axis 0 0 1, limit lower=-2.9671 upper=2.9671 effort=12 velocity=2.6100
